File: hardware/mcuderive/monezor.kicad_pcb (KiCad board)
At the start: 2 copper layers, 31.8 x 57.8 mm, 57 parts, among them J1 Conn_01x06, J2 USB_C_Receptacle, J3 Conn_01x07, SW1 SW_Push, SW2 SW_Push, U1 ATAES132A, U2 STM32F205RET6, U3 ATECC508A, U4 MCP1703A-3302_SOT23, U5 ATECC108A, U6 ATSHA204A, U7 OLED_128x64, Y1 8MHz

Commit message: version 0.2.0 initial
Parts:
- removed C1: 22p, Capacitors_SMD:C_0805
- removed C11: 100n, smd_0805_C_bottom:SMD_C_0805_bottom
- removed C15, C18, C19, C20: 2u2, smd_0805_C_bottom:SMD_C_0805_bottom
- removed U7: OLED_128x64, oled_128_x_64:oled_display128x64_bottom
- removed Y1: 8MHz, trezor_footprints:Crystal_HC52-8mm_Vertical
- added LOGO1: LOGO, monezor_footprints:xmr_logo, F.Cu at (215.9, 117.6)
- added R10: 1k, monezor_footprints:SMD_0805, F.Cu at (225.0, 98.4)
- added R9: 10k, monezor_footprints:SMD_0805, F.Cu at (226.9, 79.1)
- added S3J1: solder_jumper_3pin, monezor_footprints:solder_jumper_3pin_tht_2.54, F.Cu at (203.4, 76.4)
- added S3J2: solder_jumper_3pin, monezor_footprints:solder_jumper_3pin_tht_2.54, F.Cu at (228.4, 76.4)
- added SJ9: solder_jumper, monezor_footprints:solder_jumper, F.Cu at (230.5, 103.5)
- added X1: SG-8002JC, monezor_footprints:Oscillator_SMD_IQD_IQXO70-4pin_7.5x5.0mm, F.Cu at (225.7, 92.6)
- C10, C12, C13, C14, C16, C17, C3, C5, C7: footprint Capacitors_SMD:C_0805 -> monezor_footprints:SMD_0805
- C2: value 22p -> 15p; footprint Capacitors_SMD:C_0805 -> monezor_footprints:SMD_0805
- C4, C6, C8, C9: footprint smd_0805_C_bottom:SMD_C_0805_bottom -> monezor_footprints:SMD_0805_bottom
- D1: footprint Diodes_SMD:D_0805 -> monezor_footprints:D_SOD-523
- F1: footprint Diodes_SMD:D_0805 -> monezor_footprints:SMD_0805
- J1: value Conn_01x06 -> Programmer; footprint Pin_Headers:Pin_Header_Straight_1x06_Pitch2.54mm -> monezor_footprints:Pin_Header_Straight_1x06_Pitch2.54mm
- J2: footprint Connectors_USB:USB_C_Receptacle_Amphenol_12401548E4-2A -> monezor_footprints:USB_C_Receptacle_Amphenol_12401548E4-2A
- J3: value Conn_01x07 -> Display_module; footprint Pin_Headers:Pin_Header_Straight_1x07_Pitch2.54mm -> monezor_footprints:Pin_Header_Straight_1x07_Pitch2.54mm
- R1, R2, R3, R4, R5, R6, R7: footprint Resistors_SMD:R_0805 -> monezor_footprints:SMD_0805
- R8: value 390k -> 10k; footprint labka_footprints:SMD_0805_bottom -> monezor_footprints:SMD_0805
- SJ1, SJ2, SJ3, SJ4, SJ5, SJ6, SJ7, SJ8: footprint solderjumper_bottom:SMD_C_0805_bottom -> monezor_footprints:solderjumper_bottom
- SW1, SW2: footprint Buttons_Switches_SMD:SW_SPST_EVPBF -> monezor_footprints:BUTTON_SWITCH_SW_SPST_EVPBF
- TP1, TP2, TP3, TP4, TP5, TP6: footprint Pin_Headers:Pin_Header_Straight_1x01_Pitch1.00mm -> monezor_footprints:Test_Point_THT
- U1, U3, U5, U6: footprint soic8_bottom:SOIC-8_bottom_3.9x4.9mm_Pitch1.27mm -> monezor_footprints:SO-8_3.9x4.9mm_Pitch1.27mm_bottom
- U2: footprint Housings_QFP:TQFP-64_10x10mm_Pitch0.5mm -> monezor_footprints:TQFP-64_10x10mm_Pitch0.5mm
- U4: footprint TO_SOT_Packages_SMD:SOT-23 -> monezor_footprints:SOT-23
- moved R8 15.6 mm to (203.0, 81.4), turned to 270 degrees
- moved C3 2.83 mm to (222.1, 100.1), turned to 270 degrees
- moved TP5 2.54 mm to (230.1, 106.9)
- moved TP4 2.16 mm to (201.7, 107.3)
- moved C2 1.80 mm to (225.7, 87.2), turned to 180 degrees
- moved R4 0.48 mm to (210.8, 100.1)
- moved R1 0.47 mm to (207.9, 102.6)
Connections:
- C2 pad 1: Net-(C2-Pad1) -> GND
- C2 pad 2: GND -> Net-(C2-Pad2)
- J2 pad A10: (no net) -> Net-(J2-PadA10)
- J2 pad A11: (no net) -> Net-(J2-PadA11)
- J2 pad A2: (no net) -> Net-(J2-PadA2)
- J2 pad A3: (no net) -> Net-(J2-PadA3)
- J2 pad A5: (no net) -> Net-(J2-PadA5)
- J2 pad A8: (no net) -> Net-(J2-PadA8)
- J2 pad B10: (no net) -> Net-(J2-PadB10)
- J2 pad B11: (no net) -> Net-(J2-PadB11)
- J2 pad B2: (no net) -> Net-(J2-PadB2)
- J2 pad B3: (no net) -> Net-(J2-PadB3)
- J2 pad B5: (no net) -> Net-(J2-PadB5)
- J2 pad B8: (no net) -> Net-(J2-PadB8)
- R8 pad 2: GND -> BOOT0
- U1 pad 3: (no net) -> Net-(U1-Pad3)
- U1 pad 7: (no net) -> Net-(U1-Pad7)
- U2 pad 11: (no net) -> Net-(U2-Pad11)
- U2 pad 14: (no net) -> Net-(U2-Pad14)
- U2 pad 15: (no net) -> Net-(U2-Pad15)
- U2 pad 16: (no net) -> Net-(U2-Pad16)
- U2 pad 17: (no net) -> Net-(U2-Pad17)
- U2 pad 2: (no net) -> Net-(U2-Pad2)
- U2 pad 22: (no net) -> Net-(U2-Pad22)
- U2 pad 24: (no net) -> Net-(U2-Pad24)
- U2 pad 28: (no net) -> BOOT1
- U2 pad 29: (no net) -> Net-(U2-Pad29)
- U2 pad 3: (no net) -> Net-(U2-Pad3)
- U2 pad 30: (no net) -> Net-(U2-Pad30)
- U2 pad 33: (no net) -> Net-(U2-Pad33)
- U2 pad 34: (no net) -> Net-(U2-Pad34)
- U2 pad 35: (no net) -> Net-(U2-Pad35)
- U2 pad 36: (no net) -> Net-(U2-Pad36)
- U2 pad 37: (no net) -> Net-(U2-Pad37)
- U2 pad 38: (no net) -> Net-(U2-Pad38)
- U2 pad 39: (no net) -> Net-(U2-Pad39)
- U2 pad 4: (no net) -> Net-(U2-Pad4)
- U2 pad 40: (no net) -> Net-(U2-Pad40)
- U2 pad 41: (no net) -> Net-(U2-Pad41)
- U2 pad 43: (no net) -> Net-(U2-Pad43)
- U2 pad 5: Net-(C1-Pad1) -> Net-(C2-Pad2)
- U2 pad 50: (no net) -> Net-(U2-Pad50)
- U2 pad 51: (no net) -> Net-(U2-Pad51)
- U2 pad 52: (no net) -> Net-(U2-Pad52)
- U2 pad 53: (no net) -> Net-(U2-Pad53)
- U2 pad 54: (no net) -> Net-(U2-Pad54)
- U2 pad 56: (no net) -> Net-(U2-Pad56)
- U2 pad 57: (no net) -> Net-(U2-Pad57)
- U2 pad 6: Net-(C2-Pad1) -> GND
- U2 pad 60: GND -> BOOT0
- U2 pad 61: (no net) -> Net-(U2-Pad61)
- U2 pad 62: (no net) -> Net-(U2-Pad62)
- U2 pad 8: (no net) -> Net-(U2-Pad8)
- U2 pad 9: (no net) -> Net-(U2-Pad9)
- U3 pad 1: (no net) -> Net-(U3-Pad1)
- U3 pad 2: (no net) -> Net-(U3-Pad2)
- U3 pad 3: (no net) -> Net-(U3-Pad3)
- U3 pad 7: (no net) -> Net-(U3-Pad7)
- U5 pad 1: (no net) -> Net-(U5-Pad1)
- U5 pad 2: (no net) -> Net-(U5-Pad2)
- U5 pad 3: (no net) -> Net-(U5-Pad3)
- U5 pad 7: (no net) -> Net-(U5-Pad7)
- U6 pad 1: (no net) -> Net-(U6-Pad1)
- U6 pad 2: (no net) -> Net-(U6-Pad2)
- U6 pad 3: (no net) -> Net-(U6-Pad3)
- U6 pad 7: (no net) -> Net-(U6-Pad7)
Routing:
- net BOOT0: track 0.00 -> 25.4 mm, vias 0 -> 2
- net BOOT1: track 0.00 -> 21.6 mm, vias 0 -> 2
- net GND: track 93.9 -> 75.6 mm, vias 3 -> 14
- net PA_7: track 25.2 -> 15.0 mm
- net PB_0: track 32.6 -> 22.7 mm
- net Net-(C2-Pad2): track 0.00 -> 9.07 mm
- net PA_4: track 23.3 -> 14.6 mm
- net Net-(C2-Pad1): track 8.11 -> 0.00 mm
- net Net-(C1-Pad1): track 7.03 -> 0.00 mm
- net Net-(C15-Pad2): track 6.70 -> 0.00 mm
- net Net-(C11-Pad2): track 6.64 -> 0.00 mm
- net PB_1: track 26.2 -> 21.3 mm
- net PA_5: track 15.1 -> 10.4 mm
- net Net-(R10-Pad2): track 0.00 -> 4.57 mm
- net RST: track 19.2 -> 23.3 mm
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Other:
- board size 31.8 x 57.8 mm -> 31.8 x 47.7 mm
- board text added: "Julian Candy"
- board text added: "MONEZOR"
- board text added: "edition JC0"
- board text added: "v0.2.0 (i_a)"
- board text removed: "MCUdev 0.1"
- board text removed: "i_a"
