File: hardware/mcuderive/monezor.sch (KiCad schematic (older format))
At the start: 57 parts, among them J1 Conn_01x06, J2 USB_C_Receptacle, J3 Conn_01x07, SW1 SW_Push, SW2 SW_Push, U1 ATAES132A, U2 STM32F205RET6, U3 ATECC508A, U4 MCP1703A-3302_SOT23, U5 ATECC108A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

Commit message: version 0.2.0 initial
Parts:
- removed C1: 22p, Capacitors_SMD:C_0805, symbol C
- removed C11: 100n, smd_0805_C_bottom:SMD_C_0805_bottom, symbol C
- removed C15, C18, C19, C20: 2u2, smd_0805_C_bottom:SMD_C_0805_bottom, symbol C
- removed U7: OLED_128x64, oled_128_x_64:oled_display128x64_bottom, symbol OLED_128x64
- removed Y1: 8MHz, trezor_footprints:Crystal_HC52-8mm_Vertical, symbol Crystal
- added LOGO1: LOGO, monezor_footprints:xmr_logo, symbol LOGO
- added R10: 1k, monezor_footprints:SMD_0805, symbol R
- added R9: 10k, monezor_footprints:SMD_0805, symbol R
- added S3J1, S3J2: solder_jumper_3pin, monezor_footprints:solder_jumper_3pin_tht_2.54, symbol solder_jumper_3pin
- added SJ9: solder_jumper, monezor_footprints:solder_jumper, symbol solder_jumper
- added X1: SG-8002JC, monezor_footprints:Oscillator_SMD_IQD_IQXO70-4pin_7.5x5.0mm, symbol SG-8002JC
- C10, C12, C13, C14, C16, C17, C3, C5, C7: footprint Capacitors_SMD:C_0805 -> monezor_footprints:SMD_0805
- C2: value 22p -> 15p; footprint Capacitors_SMD:C_0805 -> monezor_footprints:SMD_0805
- C4, C6, C8, C9: footprint smd_0805_C_bottom:SMD_C_0805_bottom -> monezor_footprints:SMD_0805_bottom
- D1: footprint Diodes_SMD:D_0805 -> monezor_footprints:D_SOD-523
- F1: footprint Diodes_SMD:D_0805 -> monezor_footprints:SMD_0805
- J1: value Conn_01x06 -> Programmer; footprint Pin_Headers:Pin_Header_Straight_1x06_Pitch2.54mm -> monezor_footprints:Pin_Header_Straight_1x06_Pitch2.54mm
- J2: footprint Connectors_USB:USB_C_Receptacle_Amphenol_12401548E4-2A -> monezor_footprints:USB_C_Receptacle_Amphenol_12401548E4-2A
- J3: value Conn_01x07 -> Display_module; footprint Pin_Headers:Pin_Header_Straight_1x07_Pitch2.54mm -> monezor_footprints:Pin_Header_Straight_1x07_Pitch2.54mm
- R1, R2, R3, R4, R5, R6, R7: footprint Resistors_SMD:R_0805 -> monezor_footprints:SMD_0805
- R8: value 390k -> 10k; footprint labka_footprints:SMD_0805_bottom -> monezor_footprints:SMD_0805
- SJ1, SJ2, SJ3, SJ4, SJ5, SJ6, SJ7, SJ8: footprint solderjumper_bottom:SMD_C_0805_bottom -> monezor_footprints:solderjumper_bottom
- SW1, SW2: footprint Buttons_Switches_SMD:SW_SPST_EVPBF -> monezor_footprints:BUTTON_SWITCH_SW_SPST_EVPBF
- TP1, TP2, TP3, TP4, TP5, TP6: footprint Pin_Headers:Pin_Header_Straight_1x01_Pitch1.00mm -> monezor_footprints:Test_Point_THT
- U1, U3, U5, U6: footprint soic8_bottom:SOIC-8_bottom_3.9x4.9mm_Pitch1.27mm -> monezor_footprints:SO-8_3.9x4.9mm_Pitch1.27mm_bottom
- U2: footprint Housings_QFP:TQFP-64_10x10mm_Pitch0.5mm -> monezor_footprints:TQFP-64_10x10mm_Pitch0.5mm
- U4: footprint TO_SOT_Packages_SMD:SOT-23 -> monezor_footprints:SOT-23
Connections:
- net +3V3: now also R10.1, S3J1.3, S3J2.3, X1.4 (V+)
- net GND: now also C2.1, U2.6 (osc_out), S3J1.1, S3J2.1, SJ9.1, X1.2 (GND); no longer C2.2, R8.2, U2.60 (boot0)
- net RST: now also SJ9.2
- net BOOT1: now reaches U2.28 (pb2)
- net BOOT1: now also R9.2
- net at U2.5 (osc_in): now also C2.2, X1.3 (OUT)
- net at R8.1: now also S3J1.2
- new net: R10.2, X1.1 (OE)
- new net: R9.1, S3J2.2
- new net BOOT0: R8.2, U2.60 (boot0)
- no-connect marks 72 -> 61
Other:
- moved on the sheet: C10, C12, C13, C14, C16, C17, C2, C3, C4, C5, C6, C7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
