File: hardware/monezor/monezor.kicad_pcb (KiCad board)
At the start: 2 copper layers, 31.8 x 47.7 mm, 56 parts, among them J1 Programmer, J2 USB_C_Receptacle, J3 Display_module, SW1 SW_Push, SW2 SW_Push, U1 ATAES132A, U2 STM32F205RET6, U3 ATECC508A, U4 MCP1703A-3302_SOT23, U5 ATECC108A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

Commit message: Remaked panelization, added fiducials, generated new manufacturing data
Parts:
- added FID1: Fiducial, monezor_footprints:Fiducial_Modern_SilkscreenTop, F.Cu at (198.8, 122.6)
- added FID2: Fiducial, monezor_footprints:Fiducial_Modern_SilkscreenTop, F.Cu at (233.0, 122.6)
- added FID3: Fiducial, monezor_footprints:Fiducial_Modern_SilkscreenTop, F.Cu at (198.8, 72.4)
Changed lines of the file:
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@@
-(kicad_pcb (version 4) (host pcbnew 4.0.6)
+(kicad_pcb (version 4) (host pcbnew 4.0.7-e2-6376~58~ubuntu16.04.1)
   (general
     (links 136)
     (no_connects 0)
-    (area 191.677309 70.314285 247.118 129.065001)
+    (area 191.677309 68.51526 251.461393 129.065001)
     (thickness 1.6)
     (drawings 34)
     (tracks 566)
     (zones 0)
-    (modules 56)
+    (modules 59)
     (nets 99)
   )
@@
     (fp_line (start -1.524 1.016) (end -2.159 1.016) (layer B.Mask) (width 0.15))
   )
+  (module monezor_footprints:Fiducial_Modern_SilkscreenTop locked (layer F.Cu)
+    (at 198.755 122.6312)
+    (descr "Fiducial, Modern, Silkscreen Top, Passermarke,")
+    (tags "Fiducial, Modern, Silkscreen Top, Passermarke,")
+    (fp_text reference FID1 (at 0.03048 -4.26974) (layer F.SilkS)
+      (effects (font (size 1 1) (thickness 0.15)))
+    )
+    (fp_text value Fiducial (at 0.81026 4.18084) (layer F.Fab)
+      (effects (font (size 1 1) (thickness 0.15)))
+    )
+    (fp_circle (center 0 0) (end 1.52908 0) (layer F.SilkS) (width 0.15))
+    (fp_circle (center 0 0) (end 1.7907 0) (layer F.SilkS) (width 0.15))
+    (pad ~ smd circle (at 0 0) (size 4.8006 4.8006) (layers F.Mask)
+      (solder_mask_margin 2.99974))
+  )
+  (module monezor_footprints:Fiducial_Modern_SilkscreenTop locked (layer F.Cu)
+    (at 233.045 122.6312)
+    (descr "Fiducial, Modern, Silkscreen Top, Passermarke,")
+    (tags "Fiducial, Modern, Silkscreen Top, Passermarke,")
+    (fp_text reference FID2 (at 0.03048 -4.26974) (layer F.SilkS)
+      (effects (font (size 1 1) (thickness 0.15)))
+    )
+    (fp_text value Fiducial (at 0.81026 4.18084) (layer F.Fab)
+      (effects (font (size 1 1) (thickness 0.15)))
+    )
+    (fp_circle (center 0 0) (end 1.52908 0) (layer F.SilkS) (width 0.15))
+    (fp_circle (center 0 0) (end 1.7907 0) (layer F.SilkS) (width 0.15))
+    (pad ~ smd circle (at 0 0) (size 4.8006 4.8006) (layers F.Mask)
+      (solder_mask_margin 2.99974))
+  )
+  (module monezor_footprints:Fiducial_Modern_SilkscreenTop locked (layer F.Cu)
+    (at 198.755 72.39)
+    (descr "Fiducial, Modern, Silkscreen Top, Passermarke,")
+    (tags "Fiducial, Modern, Silkscreen Top, Passermarke,")
+    (fp_text reference FID3 (at 0.03048 -4.26974) (layer F.SilkS)
+      (effects (font (size 1 1) (thickness 0.15)))
+    )
+    (fp_text value Fiducial (at 0.81026 4.18084) (layer F.Fab)
+      (effects (font (size 1 1) (thickness 0.15)))
+    )
+    (fp_circle (center 0 0) (end 1.52908 0) (layer F.SilkS) (width 0.15))
+    (fp_circle (center 0 0) (end 1.7907 0) (layer F.SilkS) (width 0.15))
+    (pad ~ smd circle (at 0 0) (size 4.8006 4.8006) (layers F.Mask)
+      (solder_mask_margin 2.99974))
+  )
+  (dimension 47.701227 (width 0.3) (layer Dwgs.User)
+    (gr_text "47,701 mm" (at 244.961393 97.504293 270.0610178) (layer Dwgs.User)
+      (effects (font (size 1.5 1.5) (thickness 0.3)))
+    )
+    (feature1 (pts (xy 239.014 73.66) (xy 246.285992 73.652256)))
+    (feature2 (pts (xy 239.0648 121.3612) (xy 246.336792 121.353456)))
+    (crossbar (pts (xy 243.636794 121.356331) (xy 243.585994 73.655131)))
+    (arrow1a (pts (xy 243.585994 73.655131) (xy 244.173614 74.78101)))
+    (arrow1b (pts (xy 243.585994 73.655131) (xy 243.000773 74.782259)))
+    (arrow2a (pts (xy 243.636794 121.356331) (xy 244.222015 120.229203)))
+    (arrow2b (pts (xy 243.636794 121.356331) (xy 243.049174 120.230452)))
+  )
   (dimension 31.75 (width 0.3) (layer Dwgs.User)
     (gr_text "31,750 mm" (at 215.9 127.715) (layer Dwgs.User)
@@
     (arrow2b (pts (xy 200.025 126.365) (xy 201.151504 125.778579)))
   )
-  (dimension 47.752 (width 0.3) (layer Dwgs.User)
-    (gr_text "47,752 mm" (at 240.618 97.536 90) (layer Dwgs.User)
-      (effects (font (size 1.5 1.5) (thickness 0.3)))
-    )
-    (feature1 (pts (xy 236.728 73.66) (xy 241.968 73.66)))
-    (feature2 (pts (xy 236.728 121.412) (xy 241.968 121.412)))
-    (crossbar (pts (xy 239.268 121.412) (xy 239.268 73.66)))
-    (arrow1a (pts (xy 239.268 73.66) (xy 239.854421 74.786504)))
-    (arrow1b (pts (xy 239.268 73.66) (xy 238.681579 74.786504)))
-    (arrow2a (pts (xy 239.268 121.412) (xy 239.854421 120.285496)))
-    (arrow2b (pts (xy 239.268 121.412) (xy 238.681579 120.285496)))
-  )
   (gr_text "edition JC0" (at 207.01 117.475) (layer B.Mask)
