File: hardware/cloneledg/ledgblue/ledgblue.sch (KiCad schematic (older format))
At the start: 61 parts, among them J1 USB_OTG, P1 DEBUG, P2 DEBUG, P3 YL035MY2, P4 YL035MY2_TS_WURTH, SW1 WURTH 436353045816, SW2 SW-PB, U1 LD39020_3.0V, U2 STMPS2151TTR, U3 ST31G480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

Commit message: Layout has been compacted
The layout has been shrunk a bit. A pin header is used as placeholder for the antenna. NFC chip still not connected.
Parts:
- L1: footprint (none) -> Connectors:PINHEAD1-2
Changed lines of the file:
@@
 F 0 "L1" V 11000 7650 50  0000 C CNN
 F 1 "Antenna" V 11125 7650 50  0000 C CNN
-F 2 "" H 11050 7650 50  0001 C CNN
+F 2 "Connectors:PINHEAD1-2" H 11050 7650 50  0001 C CNN
 F 3 "" H 11050 7650 50  0001 C CNN
 	1    11050 7650
