File: hardware/breakneck/breakpanel.kicad_pcb (KiCad board)
At the start: 2 copper layers, 145 x 165 mm, 690 parts, among them J1 CONN_WEST, J10 GS2, J12 CONN_JTAG_6P, J15 GS2, J16 CONN_JST, J2 CONN_DEDI, J3 CONN_OLED, J4 USB_C_Receptacle, J5 CONN_SOUTH, J6 CONN_EAST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

Commit message: Corrected incompatible SE (608A) timing in ROM assistance.
This follows advice taken from Microchip case 00347747, warning against
replacing the CEC1702 ROM addendum specification of ATECC508A with the
more capable ATECC608A SE.
Parts:
- U1 (x6): value ATECC608A -> ATECC508A
Changed lines of the file:
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@@
       (effects (font (size 1 1) (thickness 0.15)))
     )
-    (fp_text value ATECC608A (at 0 2.55 180) (layer F.Fab)
+    (fp_text value ATECC508A (at 0 2.55 180) (layer F.Fab)
       (effects (font (size 1 1) (thickness 0.15)))
     )
@@
       (effects (font (size 1 1) (thickness 0.15)))
     )
-    (fp_text value ATECC608A (at 0 2.55 180) (layer F.Fab)
+    (fp_text value ATECC508A (at 0 2.55 180) (layer F.Fab)
       (effects (font (size 1 1) (thickness 0.15)))
     )
@@
       (effects (font (size 1 1) (thickness 0.15)))
     )
-    (fp_text value ATECC608A (at 0 2.55 180) (layer F.Fab)
+    (fp_text value ATECC508A (at 0 2.55 180) (layer F.Fab)
       (effects (font (size 1 1) (thickness 0.15)))
     )
@@
       (effects (font (size 1 1) (thickness 0.15)))
     )
-    (fp_text value ATECC608A (at 0 2.55 180) (layer F.Fab)
+    (fp_text value ATECC508A (at 0 2.55 180) (layer F.Fab)
       (effects (font (size 1 1) (thickness 0.15)))
     )
@@
       (effects (font (size 1 1) (thickness 0.15)))
     )
-    (fp_text value ATECC608A (at 0 2.55 180) (layer F.Fab)
+    (fp_text value ATECC508A (at 0 2.55 180) (layer F.Fab)
       (effects (font (size 1 1) (thickness 0.15)))
     )
@@
       (effects (font (size 1 1) (thickness 0.15)))
     )
-    (fp_text value ATECC608A (at 0 2.55 180) (layer F.Fab)
+    (fp_text value ATECC508A (at 0 2.55 180) (layer F.Fab)
       (effects (font (size 1 1) (thickness 0.15)))
     )
